File: hardware/LTC4150 BOB.brd (EAGLE design)
At the start: 15.2 x 30.5 mm, 23 parts, among them U1 LTC4150

Commit message: V02 ready for prototype
Parts:
- R1: device SparkFun-Passives:0805 -> SparkFun-Passives:1206
- R4, R8: value 75K -> 47K
- R5, R7: value 3K -> 3.3K
- moved JP2 2.54 mm to (1.27, 16.5), turned to 90 degrees
- moved JP3 2.54 mm to (14.0, 19.1), turned to 270 degrees
Connections:
- net !CLR!: now also JP4.5; no longer JP4.3
- net !SHDN!: now also JP4.6; no longer JP4.5
- net GND: now also JP4.4; no longer JP4.6
- net POL: now also JP4.3; no longer JP4.4
Routing:
- net !SHDN!: track 20.7 -> 17.3 mm, vias 1 -> 2
- net !CLR!: track 20.2 -> 17.4 mm, vias 0 -> 1
- net POL: track 12.1 -> 13.2 mm
- net OUT: track 22.4 -> 21.9 mm
- net IN: track 14.8 -> 14.3 mm
- net GND: vias 4 -> 7
Other:
- board text added: "+IN"
- board text added: "-OUT"
- board text added: "V02"
- board text removed: "+OUT"
- board text removed: "-IN"
- board text removed: "V01"
